Commit message: second commit

File: telemarketing_description/urdf/gazebo.xacro (robot description, xacro)
@@ -1,6 +1,58 @@
 <?xml version="1.0" ?>
-<robot name="Telemarket" xmlns:xacro="http://www.ros.org/wiki/xacro">
+<robot name="Telemarketing" xmlns:xacro="http://www.ros.org/wiki/xacro">
   <gazebo reference="base_link">
-    <material>Gazebo/Orange</material>
+    <material>Gazebo/Grey</material>
+  </gazebo>
+  <gazebo reference="left_wheel">
+    <mu1>0.9</mu1>
+    <mu2>0.9</mu2>
+    <kp>500000.0</kp>
+    <kd>10.0</kd>
+    <minDepth>0.001</minDepth>
+    <maxVel>0.1</maxVel>
+    <fdir1>1 0 0</fdir1>
+    <material>Gazebo/FlatBlack</material>
+  </gazebo>
+  <gazebo reference="right_wheel">
+    <mu1>0.9</mu1>
+    <mu2>0.9</mu2>
+    <kp>500000.0</kp>
+    <kd>10.0</kd>
+    <minDepth>0.001</minDepth>
+    <maxVel>0.1</maxVel>
+    <fdir1>1 0 0</fdir1>
+    <material>Gazebo/FlatBlack</material>
+  </gazebo>
+<!--
+  <gazebo>
+    <plugin name="gazebo_ros_control" filename="libgazebo_ros_control.so">
+      <robotSimType>gazebo_ros_control/DefaultRobotHWSim</robotSimType>
+      <robotNamespace>/thesis</robotNamespace>
+      <legacyModeNS>true</legacyModeNS>
+    </plugin>
+  </gazebo>-->
+  <gazebo>
+    <plugin name='differential_drive_controller' filename='libgazebo_ros_diff_drive.so'>
+      <alwaysOn>true</alwaysOn>
+      <leftJoint>l_wheel_joint</leftJoint>
+      <rightJoint>r_wheel_joint</rightJoint>
+      <updateRate>100</updateRate>
+      <robotBaseFrame>base_link</robotBaseFrame>
+      <covariance_x>0.0001</covariance_x>
+      <covariance_y>0.0001</covariance_y>
+      <covariance_yaw>0.01</covariance_yaw>
+      <wheelSeparation>0.6910</wheelSeparation>
+      <wheelDiameter>0.32766</wheelDiameter>
+      <torque>100</torque>
+      <wheelAcceleration>0.1</wheelAcceleration>
+      <commandTopic>cmd_vel</commandTopic>
+      <odometryTopic>odom</odometryTopic>
+      <odometryFrame>odom</odometryFrame>
+      <broadcastTF>true</broadcastTF>
+      <publishWheelTF>true</publishWheelTF>
+      <publishOdom>true</publishOdom>
+      <publishWheelJointState>true</publishWheelJointState>
+      <legacyMode>false</legacyMode>
+    </plugin>
   </gazebo>
 </robot>

File: telemarketing_description/urdf/telemarketing.xacro (robot description, xacro)
@@ -20,10 +20,10 @@
   <!-- Robot description -->
   <m_link_mesh name="base_link"
-              origin_rpy="0 0 0" origin_xyz="0 0 0.2355"
+              origin_rpy="0 1.5708 3.1416" origin_xyz="0 0 0.2355"
               mass="80"
-              ixx="0.8837" ixy="0" ixz="0"
-              iyy="2.6409" iyz="0"
-              izz="3.0534"
-              material="orange"
+              ixx="1177287.158" ixy="-246402.075" ixz="-453961.379"
+              iyy="13057357.025" iyz="-55693.992"
+              izz="13181014.451"
+              material="grey"
               meshfile="package://telemarket_description/meshes/main_frame.stl"
               meshscale="0.010335 0.010335 0.010335" />

Commit message: third commit

File: telemarketing_description/urdf/gazebo.xacro (robot description, xacro)
@@ -2,9 +2,9 @@
 <robot name="Telemarketing" xmlns:xacro="http://www.ros.org/wiki/xacro">
   <gazebo reference="base_link">
-    <material>Gazebo/Grey</material>
+    <material>Gazebo/White</material>
   </gazebo>
-  <gazebo reference="left_wheel">
-    <mu1>0.9</mu1>
-    <mu2>0.9</mu2>
+  <gazebo reference="r_dwheel">
+    <mu1>1.0</mu1>
+    <mu2>1.0</mu2>
     <kp>500000.0</kp>
     <kd>10.0</kd>
@@ -14,7 +14,47 @@
     <material>Gazebo/FlatBlack</material>
   </gazebo>
-  <gazebo reference="right_wheel">
-    <mu1>0.9</mu1>
-    <mu2>0.9</mu2>
+  <gazebo reference="l_dwheel">
+    <mu1>1.0</mu1>
+    <mu2>1.0</mu2>
+    <kp>500000.0</kp>
+    <kd>10.0</kd>
+    <minDepth>0.001</minDepth>
+    <maxVel>0.1</maxVel>
+    <fdir1>1 0 0</fdir1>
+    <material>Gazebo/FlatBlack</material>
+  </gazebo>
+  <gazebo reference="fr_cwheel">
+    <mu1>0.0</mu1>
+    <mu2>0.0</mu2>
+    <kp>500000.0</kp>
+    <kd>10.0</kd>
+    <minDepth>0.001</minDepth>
+    <maxVel>0.1</maxVel>
+    <fdir1>1 0 0</fdir1>
+    <material>Gazebo/FlatBlack</material>
+  </gazebo>
+  <gazebo reference="fl_cwheel">
+    <mu1>0.0</mu1>
+    <mu2>0.0</mu2>
+    <kp>500000.0</kp>
+    <kd>10.0</kd>
+    <minDepth>0.001</minDepth>
+    <maxVel>0.1</maxVel>
+    <fdir1>1 0 0</fdir1>
+    <material>Gazebo/FlatBlack</material>
+  </gazebo>
+  <gazebo reference="br_cwheel">
+    <mu1>0.0</mu1>
+    <mu2>0.0</mu2>
+    <kp>500000.0</kp>
+    <kd>10.0</kd>
+    <minDepth>0.001</minDepth>
+    <maxVel>0.1</maxVel>
+    <fdir1>1 0 0</fdir1>
+    <material>Gazebo/FlatBlack</material>
+  </gazebo>
+  <gazebo reference="bl_cwheel">
+    <mu1>0.0</mu1>
+    <mu2>0.0</mu2>
     <kp>500000.0</kp>
     <kd>10.0</kd>
@@ -34,24 +74,24 @@
   <gazebo>
     <plugin name='differential_drive_controller' filename='libgazebo_ros_diff_drive.so'>
-      <alwaysOn>true</alwaysOn>
-      <leftJoint>l_wheel_joint</leftJoint>
-      <rightJoint>r_wheel_joint</rightJoint>
       <updateRate>100</updateRate>
-      <robotBaseFrame>base_link</robotBaseFrame>
-      <covariance_x>0.0001</covariance_x>
-      <covariance_y>0.0001</covariance_y>
-      <covariance_yaw>0.01</covariance_yaw>
-      <wheelSeparation>0.6910</wheelSeparation>
-      <wheelDiameter>0.32766</wheelDiameter>
-      <torque>100</torque>
+      <leftJoint>l_dwheel_joint</leftJoint>
+      <rightJoint>r_dwheel_joint</rightJoint>
+      <wheelSeparation>0.3219</wheelSeparation>
+      <wheelDiameter>0.2032</wheelDiameter>
       <wheelAcceleration>0.1</wheelAcceleration>
+      <wheelTorque>40</wheelTorque>
       <commandTopic>cmd_vel</commandTopic>
       <odometryTopic>odom</odometryTopic>
       <odometryFrame>odom</odometryFrame>
-      <broadcastTF>true</broadcastTF>
+      <robotBaseFrame>base_link</robotBaseFrame>
       <publishWheelTF>true</publishWheelTF>
       <publishOdom>true</publishOdom>
       <publishWheelJointState>true</publishWheelJointState>
       <legacyMode>false</legacyMode>
+      <alwaysOn>true</alwaysOn>
+      <covariance_x>0.0001</covariance_x>
+      <covariance_y>0.0001</covariance_y>
+      <covariance_yaw>0.01</covariance_yaw>
+      <broadcastTF>true</broadcastTF>
     </plugin>
   </gazebo>

File: telemarketing_description/urdf/telemarketing.xacro (robot description, xacro)
@@ -1,6 +1,6 @@
 <?xml version="1.0" ?>
-<robot name="Telemarket" xmlns:xacro="http://www.ros.org/wiki/xacro">
-  <xacro:include filename="$(find telemarket_description)/urdf/links_joints.xacro" />
-  <xacro:include filename="$(find telemarket_description)/urdf/gazebo.xacro" />
+<robot name="Telemarketing" xmlns:xacro="http://www.ros.org/wiki/xacro">
+  <xacro:include filename="$(find telemarketing_description)/urdf/links_joints.xacro" />
+  <xacro:include filename="$(find telemarketing_description)/urdf/gazebo.xacro" />
   <material name="white">
     <color rgba="1 1 1 1"/>
@@ -20,11 +20,28 @@
   <!-- Robot description -->
   <m_link_mesh name="base_link"
-              origin_rpy="0 1.5708 3.1416" origin_xyz="0 0 0.2355"
-              mass="80"
+              origin_rpy="0 0 0" origin_xyz="0 0 0"
+              mass="1"
               ixx="1177287.158" ixy="-246402.075" ixz="-453961.379"
               iyy="13057357.025" iyz="-55693.992"
               izz="13181014.451"
-              material="grey"
-              meshfile="package://telemarket_description/meshes/main_frame.stl"
+              material="white"
+              meshfile="package://telemarketing_description/meshes/main_frame.stl"
               meshscale="0.010335 0.010335 0.010335" />
+<!--
+  <joint name="l_dwheel_joint" type="continuous">
+      <parent link="base_link"/>
+      <child link="l_dwheel"/>
+      <origin xyz="0.311 0.3455 0.1016" rpy="0.0 0.0 0"/>
+      <axis xyz="0 1 0"/>
+  </joint>
+  <m_link_mesh name="l_dwheel"
+              origin_rpy="0 0 0" origin_xyz="0 0 0"
+              mass="10"
+              ixx="0.1798" ixy="0" ixz="0"
+              iyy="0.1081" iyz="0"
+              izz="0.1798"
+              material="black"
+              meshfile="package://telemarketing_description/meshes/main_wheel.stl"
+              meshscale="0.010335 0.010335 0.010335" />
+-->
 </robot>

Commit message: Update several packages

File: telemarketing_description/urdf/gazebo.xacro (robot description, xacro)
@@ -1,7 +1,9 @@
 <?xml version="1.0" ?>
 <robot name="Telemarketing" xmlns:xacro="http://www.ros.org/wiki/xacro">
+  <!-- Base link -->
   <gazebo reference="base_link">
     <material>Gazebo/White</material>
   </gazebo>
+  <!-- Right drive wheel -->
   <gazebo reference="r_dwheel">
     <mu1>1.0</mu1>
@@ -14,4 +16,5 @@
     <material>Gazebo/FlatBlack</material>
   </gazebo>
+  <!-- Left drive wheel -->
   <gazebo reference="l_dwheel">
     <mu1>1.0</mu1>
@@ -24,4 +27,5 @@
     <material>Gazebo/FlatBlack</material>
   </gazebo>
+  <!-- Front right caster wheel -->
   <gazebo reference="fr_cwheel">
     <mu1>0.0</mu1>
@@ -34,4 +38,5 @@
     <material>Gazebo/FlatBlack</material>
   </gazebo>
+  <!-- Front left caster wheel -->
   <gazebo reference="fl_cwheel">
     <mu1>0.0</mu1>
@@ -44,4 +49,5 @@
     <material>Gazebo/FlatBlack</material>
   </gazebo>
+  <!-- Back right caster wheel -->
   <gazebo reference="br_cwheel">
     <mu1>0.0</mu1>
@@ -54,4 +60,5 @@
     <material>Gazebo/FlatBlack</material>
   </gazebo>
+  <!-- Back left caster wheel -->
   <gazebo reference="bl_cwheel">
     <mu1>0.0</mu1>
@@ -64,14 +71,8 @@
     <material>Gazebo/FlatBlack</material>
   </gazebo>
-<!--
-  <gazebo>
-    <plugin name="gazebo_ros_control" filename="libgazebo_ros_control.so">
-      <robotSimType>gazebo_ros_control/DefaultRobotHWSim</robotSimType>
-      <robotNamespace>/thesis</robotNamespace>
-      <legacyModeNS>true</legacyModeNS>
-    </plugin>
-  </gazebo>-->
+  <!-- Plugin for differential drive controller -->
   <gazebo>
     <plugin name='differential_drive_controller' filename='libgazebo_ros_diff_drive.so'>
+      <!--<alwaysOn>true</alwaysOn>-->
       <updateRate>100</updateRate>
       <leftJoint>l_dwheel_joint</leftJoint>
@@ -84,15 +85,44 @@
       <odometryTopic>odom</odometryTopic>
       <odometryFrame>odom</odometryFrame>
-      <robotBaseFrame>base_link</robotBaseFrame>
+      <robotBaseFrame>base_footprint</robotBaseFrame>
       <publishWheelTF>true</publishWheelTF>
       <publishOdom>true</publishOdom>
+      <robotBaseFrame>base</robotBaseFrame>
       <publishWheelJointState>true</publishWheelJointState>
       <legacyMode>false</legacyMode>
-      <alwaysOn>true</alwaysOn>
-      <covariance_x>0.0001</covariance_x>
-      <covariance_y>0.0001</covariance_y>
-      <covariance_yaw>0.01</covariance_yaw>
-      <broadcastTF>true</broadcastTF>
     </plugin>
   </gazebo>
+  <!-- LiDAR -->
+  <gazebo reference="lidar_link">
+    <material>Gazebo/Blue</material>
+    <sensor type="ray" name="hokuyo_sensor">
+      <pose>0 0 0 1.5708 0 1.5708</pose>
+      <visualize>true</visualize>
+      <update_rate>40</update_rate>
+      <ray>
+        <scan>
+          <horizontal>
+            <samples>1080</samples>
+            <resolution>0.25</resolution>
+            <min_angle>-2.3562</min_angle>
+            <max_angle>2.3562</max_angle>
+          </horizontal>
+        </scan>
+        <range>
+          <min>0.20</min>
+          <max>16.0</max>
+          <resolution>0.001</resolution>
+        </range>
+        <noise>
+          <type>gaussian</type>
+          <mean>0.0</mean>
+          <stddev>0.01</stddev>
+        </noise>
+      </ray>
+      <plugin name="gazebo_ros_head_hokuyo_controller" filename="libgazebo_ros_laser.so">
+        <topicName>/laser_scan</topicName>
+        <frameName>lidar_link</frameName>
+      </plugin>
+    </sensor>
+  </gazebo>
 </robot>

File: telemarketing_description/urdf/telemarketing.xacro (robot description, xacro)
@@ -13,10 +13,10 @@
   </material>
   <material name="grey">
-    <color rgba="0.332 0.332 0.332 1"/>
+    <color rgba="0.750 0.750 0.750 1"/>
   </material>
   <material name="orange">
     <color rgba="0.949 0.361 0.098 1"/>
   </material>
-  <!-- Robot description 0.311 0.3455 0.1016 -->
+  <!-- Robot description -->
   <m_link_mesh name="base_link"
               origin_rpy="0 1.5708 3.1416" origin_xyz="0 0.158 0.5"
@@ -25,11 +25,26 @@
               iyy="13057357.025" iyz="-55693.992"
               izz="13181014.451"
-              material="white"
+              material="grey"
               meshfile="package://telemarketing_description/meshes/main_frame.stl"
+              meshscale="0.010335 0.010335 0.010335" />
+  <joint name="r_dwheel_joint" type="continuous">
+      <parent link="base_link"/>
+      <child link="r_dwheel"/>
+      <origin xyz="-0.026 -0.174 0.661" rpy="1.5708 0.0 0"/>
+      <axis xyz="0 1 0"/>
+  </joint>
+  <m_link_mesh name="r_dwheel"
+              origin_rpy="0 0 0" origin_xyz="0 0 0"
+              mass="10"
+              ixx="0.1798" ixy="0" ixz="0"
+              iyy="0.1081" iyz="0"
+              izz="0.1798"
+              material="black"
+              meshfile="package://telemarketing_description/meshes/main_wheel.stl"
               meshscale="0.010335 0.010335 0.010335" />
   <joint name="l_dwheel_joint" type="continuous">
       <parent link="base_link"/>
       <child link="l_dwheel"/>
-      <origin xyz="-0.065 -0.144 0.661" rpy="0.0 0.0 0"/>
+      <origin xyz="-0.007 0.169 0.661" rpy="1.5708 0.0 0"/>
       <axis xyz="0 1 0"/>
   </joint>
@@ -43,3 +58,63 @@
               meshfile="package://telemarketing_description/meshes/main_wheel.stl"
               meshscale="0.010335 0.010335 0.010335" />
+  <joint name="fr_cwheel_joint" type="continuous">
+      <parent link="base_link"/>
+      <child link="fr_cwheel"/>
+      <origin xyz="0.165 -0.186 0.609" rpy="1.5708 0.0 0"/>
+      <axis xyz="0 1 0"/>
+  </joint>
+  <m_link_mesh name="fr_cwheel"
+              origin_rpy="0 0 0" origin_xyz="0 0 0"
+              mass="10"
+              ixx="0.1798" ixy="0" ixz="0"
+              iyy="0.1081" iyz="0"
+              izz="0.1798"
+              material="black"
+              meshfile="package://telemarketing_description/meshes/caster_wheel.stl"
+              meshscale="0.010335 0.010335 0.010335" />
+  <joint name="fl_cwheel_joint" type="continuous">
+      <parent link="base_link"/>
+      <child link="fl_cwheel"/>
+      <origin xyz="0.165 0.181 0.609" rpy="1.5708 0.0 0"/>
+      <axis xyz="0 1 0"/>
+  </joint>
+  <m_link_mesh name="fl_cwheel"
+              origin_rpy="0 0 0" origin_xyz="0 0 0"
+              mass="10"
+              ixx="0.1798" ixy="0" ixz="0"
+              iyy="0.1081" iyz="0"
+              izz="0.1798"
+              material="black"
+              meshfile="package://telemarketing_description/meshes/caster_wheel.stl"
+              meshscale="0.010335 0.010335 0.010335" />
+  <joint name="br_cwheel_joint" type="continuous">
+      <parent link="base_link"/>
+      <child link="br_cwheel"/>
+      <origin xyz="-0.199 -0.186 0.609" rpy="1.5708 0.0 0"/>
+      <axis xyz="0 1 0"/>
+  </joint>
+  <m_link_mesh name="br_cwheel"
+              origin_rpy="0 0 0" origin_xyz="0 0 0"
+              mass="10"
+              ixx="0.1798" ixy="0" ixz="0"
+              iyy="0.1081" iyz="0"
+              izz="0.1798"
+              material="black"
+              meshfile="package://telemarketing_description/meshes/caster_wheel.stl"
+              meshscale="0.010335 0.010335 0.010335" />
+  <joint name="bl_cwheel_joint" type="continuous">
+      <parent link="base_link"/>
+      <child link="bl_cwheel"/>
+      <origin xyz="-0.199 0.181 0.609" rpy="1.5708 0.0 0"/>
+      <axis xyz="0 1 0"/>
+  </joint>
+  <m_link_mesh name="bl_cwheel"
+              origin_rpy="0 0 0" origin_xyz="0 0 0"
+              mass="10"
+              ixx="0.1798" ixy="0" ixz="0"
+              iyy="0.1081" iyz="0"
+              izz="0.1798"
+              material="black"
+              meshfile="package://telemarketing_description/meshes/caster_wheel.stl"
+              meshscale="0.010335 0.010335 0.010335" />
 </robot>

Commit message: Update telemarketing descriptiion

File: telemarketing_description/urdf/gazebo.xacro (robot description, xacro)
@@ -94,4 +94,5 @@
   </gazebo>
   <!-- LiDAR -->
+  <!-- https://bucket-download.slamtec.com/4cc2c07b7d31bbcb62eb6183f448deb2b6b36da4/LD206_SLAMTEC_rplidar_datasheet_A2M6_v0.6_en.pdf -->
   <gazebo reference="lidar_link">
     <material>Gazebo/Blue</material>
@@ -99,12 +100,12 @@
       <pose>0 0 0 1.5708 0 1.5708</pose>
       <visualize>true</visualize>
-      <update_rate>40</update_rate>
+      <update_rate>10</update_rate>
       <ray>
         <scan>
           <horizontal>
-            <samples>1080</samples>
-            <resolution>0.25</resolution>
-            <min_angle>-2.3562</min_angle>
-            <max_angle>2.3562</max_angle>
+            <samples>400</samples>
+            <resolution>0.9</resolution>
+            <min_angle>0</min_angle>
+            <max_angle>6.2832</max_angle>
           </horizontal>
         </scan>
@@ -112,5 +113,5 @@
           <min>0.20</min>
           <max>16.0</max>
-          <resolution>0.001</resolution>
+          <resolution>0.1</resolution>
         </range>
         <noise>
@@ -126,3 +127,46 @@
     </sensor>
   </gazebo>
+  <!-- Depth camera -->
+  <gazebo reference="depth_link">
+    <material>Gazebo/Blue</material>
+    <sensor name="depth_camera" type="depth">
+      <update_rate>15</update_rate>
+      <camera>
+        <horizontal_fov>1.204277</horizontal_fov>
+        <image>
+          <width>1920</width>
+          <height>1080</height>
+          <format>R8G8B8</format>
+        </image>
+        <clip>
+          <near>0.3</near>
+          <far>3.0</far>
+        </clip>
+      </camera>
+      <plugin name="depth_link_controller" filename="libgazebo_ros_openni_kinect.so">
+        <baseline>0.05</baseline>
+        <alwaysOn>true</alwaysOn>
+        <updateRate>1.0</updateRate>
+        <cameraName>depth_camera_ir</cameraName>
+        <imageTopicName>depth_camera/color/image_raw</imageTopicName>
+        <cameraInfoTopicName>/depth_camera/color/camera_info</cameraInfoTopicName>
+        <depthImageTopicName>/depth_camera/depth/image_raw</depthImageTopicName>
+        <depthImageInfoTopicName>/depth_camera/depth/camera_info</depthImageInfoTopicName>
+        <pointCloudTopicName>/depth_camera/depth/points</pointCloudTopicName>
+        <frameName>depth_optical_link</frameName>
+        <pointCloudCutoff>0.3</pointCloudCutoff>
+        <pointCloudCutoffMax>3.0</pointCloudCutoffMax>
+        <distortionK1>0.00000001</distortionK1>
+        <distortionK2>0.00000001</distortionK2>
+        <distortionK3>0.00000001</distortionK3>
+        <distortionT1>0.00000001</distortionT1>
+        <distortionT2>0.00000001</distortionT2>
+        <CxPrime>0</CxPrime>
+        <Cx>0</Cx>
+        <Cy>0</Cy>
+        <focalLength>0</focalLength>
+        <hackBaseline>0</hackBaseline>
+      </plugin>
+    </sensor>
+  </gazebo>
 </robot>

File: telemarketing_description/urdf/telemarketing.xacro (robot description, xacro)
@@ -118,3 +118,61 @@
               meshfile="package://telemarketing_description/meshes/caster_wheel.stl"
               meshscale="0.010335 0.010335 0.010335" />
+  <joint name="lidar_joint" type="fixed">
+    <axis xyz="0 1 0" />
+    <origin xyz="0.1650 0 0.920" rpy="0 0 0"/>
+    <parent link="base_link"/>
+    <child link="lidar_link"/>
+  </joint>
+  <link name="lidar_link">
+    <collision>
+      <origin xyz="0 0 0" rpy="1.5708 0 1.5708"/>
+      <geometry>
+        <mesh filename="package://telemarketing_description/meshes/lidar.stl" scale="0.010335 0.010335 0.010335"/>
+      </geometry>
+    </collision>
+    <visual>
+      <origin xyz="0 0 0" rpy="1.5708 0 1.5708"/>
+      <geometry>
+        <mesh filename="package://telemarketing_description/meshes/lidar.stl" scale="0.010335 0.010335 0.010335"/>
+      </geometry>
+      <material name="blue"/>
+    </visual>
+    <inertial>
+      <mass value="0.370" />
+      <origin xyz="0 0 0" rpy="1.5708 0 1.5708"/>
+      <inertia ixx="1e-6" ixy="0" ixz="0" iyy="1e-6" iyz="0" izz="1e-6" />
+    </inertial>
+  </link>
+  <joint name="depth_joint" type="fixed">
+    <axis xyz="0 1 0" />
+    <origin xyz="0.165 0 1.417" rpy="0 0 0"/>
+    <parent link="base_link"/>
+    <child link="depth_link"/>
+  </joint>
+  <link name="depth_link">
+    <collision>
+      <origin xyz="0 0 0" rpy="1.3090 0 1.5708"/>
+      <geometry>
+        <mesh filename="package://telemarketing_description/meshes/depth_camera.stl" scale="0.010335 0.010335 0.010335"/>
+      </geometry>
+    </collision>
+    <visual>
+      <origin xyz="0 0 0" rpy="1.3090 0 1.5708"/>
+      <geometry>
+        <mesh filename="package://telemarketing_description/meshes/depth_camera.stl" scale="0.010335 0.010335 0.010335"/>
+      </geometry>
+      <material name="grey"/>
+    </visual>
+    <inertial>
+      <mass value="1e-5" />
+      <origin xyz="0 0 0" rpy="0 0 0"/>
+      <inertia ixx="1e-6" ixy="0" ixz="0" iyy="1e-6" iyz="0" izz="1e-6" />
+    </inertial>
+  </link>
+  <joint name="depth_optical_joint" type="fixed">
+    <origin xyz="0 0 0" rpy="-1.5708 0 -1.5708"/>
+    <parent link="depth_link"/>
+    <child link="depth_optical_link"/>
+  </joint>
+  <link name="depth_optical_link"/>
 </robot>

Commit message: Update telemarketing descriptiion

File: telemarketing_description/urdf/gazebo.xacro (robot description, xacro)
@@ -128,4 +128,6 @@
   </gazebo>
   <!-- Depth camera -->
+  <!-- https://www.intelrealsense.com/depth-camera-d435i/ -->
+  <!-- https://www.intel.com/content/dam/support/us/en/documents/emerging-technologies/intel-realsense-technology/Intel-RealSense-D400-Series-Datasheet.pdf -->
   <gazebo reference="depth_link">
     <material>Gazebo/Blue</material>

File: telemarketing_description/urdf/telemarketing.xacro (robot description, xacro)
@@ -32,5 +32,5 @@
       <child link="r_dwheel"/>
       <origin xyz="-0.026 -0.174 0.661" rpy="1.5708 0.0 0"/>
-      <axis xyz="0 1 0"/>
+      <axis xyz="0 0 -1"/>
   </joint>
   <m_link_mesh name="r_dwheel"
@@ -47,5 +47,5 @@
       <child link="l_dwheel"/>
       <origin xyz="-0.007 0.169 0.661" rpy="1.5708 0.0 0"/>
-      <axis xyz="0 1 0"/>
+      <axis xyz="0 0 -1"/>
   </joint>
   <m_link_mesh name="l_dwheel"
