Commit message: Update urdf description

File: telemarketing_description/urdf/telemarketing.xacro (robot description, xacro)
@@ -18,7 +18,7 @@
     <color rgba="0.949 0.361 0.098 1"/>
   </material>
-  <!-- Robot description -->
+  <!-- Robot description 0.311 0.3455 0.1016 -->
   <m_link_mesh name="base_link"
-              origin_rpy="0 0 0" origin_xyz="0 0 0"
+              origin_rpy="0 1.5708 3.1416" origin_xyz="0 0.158 0.5"
               mass="1"
               ixx="1177287.158" ixy="-246402.075" ixz="-453961.379"
@@ -28,9 +28,8 @@
               meshfile="package://telemarketing_description/meshes/main_frame.stl"
               meshscale="0.010335 0.010335 0.010335" />
-<!--
   <joint name="l_dwheel_joint" type="continuous">
       <parent link="base_link"/>
       <child link="l_dwheel"/>
-      <origin xyz="0.311 0.3455 0.1016" rpy="0.0 0.0 0"/>
+      <origin xyz="-0.065 -0.144 0.661" rpy="0.0 0.0 0"/>
       <axis xyz="0 1 0"/>
   </joint>
@@ -44,4 +43,3 @@
               meshfile="package://telemarketing_description/meshes/main_wheel.stl"
               meshscale="0.010335 0.010335 0.010335" />
--->
 </robot>

Commit message: Several updates

File: telemarketing_description/urdf/telemarketing.xacro (robot description, xacro)
@@ -1,178 +1,864 @@
 <?xml version="1.0" ?>
-<robot name="Telemarketing" xmlns:xacro="http://www.ros.org/wiki/xacro">
-  <xacro:include filename="$(find telemarketing_description)/urdf/links_joints.xacro" />
-  <xacro:include filename="$(find telemarketing_description)/urdf/gazebo.xacro" />
-  <material name="white">
-    <color rgba="1 1 1 1"/>
-  </material>
-  <material name="black">
-    <color rgba="0 0 0 1"/>
-  </material>
-  <material name="blue">
-    <color rgba="0 0 1 1"/>
-  </material>
-  <material name="grey">
-    <color rgba="0.750 0.750 0.750 1"/>
-  </material>
-  <material name="orange">
-    <color rgba="0.949 0.361 0.098 1"/>
-  </material>
-  <!-- Robot description -->
-  <m_link_mesh name="base_link"
-              origin_rpy="0 1.5708 3.1416" origin_xyz="0 0.158 0.5"
-              mass="1"
-              ixx="1177287.158" ixy="-246402.075" ixz="-453961.379"
-              iyy="13057357.025" iyz="-55693.992"
-              izz="13181014.451"
-              material="grey"
-              meshfile="package://telemarketing_description/meshes/main_frame.stl"
-              meshscale="0.010335 0.010335 0.010335" />
-  <joint name="r_dwheel_joint" type="continuous">
-      <parent link="base_link"/>
-      <child link="r_dwheel"/>
-      <origin xyz="-0.026 -0.174 0.661" rpy="1.5708 0.0 0"/>
-      <axis xyz="0 0 -1"/>
-  </joint>
-  <m_link_mesh name="r_dwheel"
-              origin_rpy="0 0 0" origin_xyz="0 0 0"
-              mass="10"
-              ixx="0.1798" ixy="0" ixz="0"
-              iyy="0.1081" iyz="0"
-              izz="0.1798"
-              material="black"
-              meshfile="package://telemarketing_description/meshes/main_wheel.stl"
-              meshscale="0.010335 0.010335 0.010335" />
-  <joint name="l_dwheel_joint" type="continuous">
-      <parent link="base_link"/>
-      <child link="l_dwheel"/>
-      <origin xyz="-0.007 0.169 0.661" rpy="1.5708 0.0 0"/>
-      <axis xyz="0 0 -1"/>
-  </joint>
-  <m_link_mesh name="l_dwheel"
-              origin_rpy="0 0 0" origin_xyz="0 0 0"
-              mass="10"
-              ixx="0.1798" ixy="0" ixz="0"
-              iyy="0.1081" iyz="0"
-              izz="0.1798"
-              material="black"
-              meshfile="package://telemarketing_description/meshes/main_wheel.stl"
-              meshscale="0.010335 0.010335 0.010335" />
-  <joint name="fr_cwheel_joint" type="continuous">
-      <parent link="base_link"/>
-      <child link="fr_cwheel"/>
-      <origin xyz="0.165 -0.186 0.609" rpy="1.5708 0.0 0"/>
-      <axis xyz="0 1 0"/>
-  </joint>
-  <m_link_mesh name="fr_cwheel"
-              origin_rpy="0 0 0" origin_xyz="0 0 0"
-              mass="10"
-              ixx="0.1798" ixy="0" ixz="0"
-              iyy="0.1081" iyz="0"
-              izz="0.1798"
-              material="black"
-              meshfile="package://telemarketing_description/meshes/caster_wheel.stl"
-              meshscale="0.010335 0.010335 0.010335" />
-  <joint name="fl_cwheel_joint" type="continuous">
-      <parent link="base_link"/>
-      <child link="fl_cwheel"/>
-      <origin xyz="0.165 0.181 0.609" rpy="1.5708 0.0 0"/>
-      <axis xyz="0 1 0"/>
-  </joint>
-  <m_link_mesh name="fl_cwheel"
-              origin_rpy="0 0 0" origin_xyz="0 0 0"
-              mass="10"
-              ixx="0.1798" ixy="0" ixz="0"
-              iyy="0.1081" iyz="0"
-              izz="0.1798"
-              material="black"
-              meshfile="package://telemarketing_description/meshes/caster_wheel.stl"
-              meshscale="0.010335 0.010335 0.010335" />
-  <joint name="br_cwheel_joint" type="continuous">
-      <parent link="base_link"/>
-      <child link="br_cwheel"/>
-      <origin xyz="-0.199 -0.186 0.609" rpy="1.5708 0.0 0"/>
-      <axis xyz="0 1 0"/>
-  </joint>
-  <m_link_mesh name="br_cwheel"
-              origin_rpy="0 0 0" origin_xyz="0 0 0"
-              mass="10"
-              ixx="0.1798" ixy="0" ixz="0"
-              iyy="0.1081" iyz="0"
-              izz="0.1798"
-              material="black"
-              meshfile="package://telemarketing_description/meshes/caster_wheel.stl"
-              meshscale="0.010335 0.010335 0.010335" />
-  <joint name="bl_cwheel_joint" type="continuous">
-      <parent link="base_link"/>
-      <child link="bl_cwheel"/>
-      <origin xyz="-0.199 0.181 0.609" rpy="1.5708 0.0 0"/>
-      <axis xyz="0 1 0"/>
-  </joint>
-  <m_link_mesh name="bl_cwheel"
-              origin_rpy="0 0 0" origin_xyz="0 0 0"
-              mass="10"
-              ixx="0.1798" ixy="0" ixz="0"
-              iyy="0.1081" iyz="0"
-              izz="0.1798"
-              material="black"
-              meshfile="package://telemarketing_description/meshes/caster_wheel.stl"
-              meshscale="0.010335 0.010335 0.010335" />
-  <joint name="lidar_joint" type="fixed">
-    <axis xyz="0 1 0" />
-    <origin xyz="0.1650 0 0.920" rpy="0 0 0"/>
-    <parent link="base_link"/>
-    <child link="lidar_link"/>
-  </joint>
-  <link name="lidar_link">
-    <collision>
-      <origin xyz="0 0 0" rpy="1.5708 0 1.5708"/>
-      <geometry>
-        <mesh filename="package://telemarketing_description/meshes/lidar.stl" scale="0.010335 0.010335 0.010335"/>
-      </geometry>
-    </collision>
-    <visual>
-      <origin xyz="0 0 0" rpy="1.5708 0 1.5708"/>
-      <geometry>
-        <mesh filename="package://telemarketing_description/meshes/lidar.stl" scale="0.010335 0.010335 0.010335"/>
-      </geometry>
-      <material name="blue"/>
-    </visual>
-    <inertial>
-      <mass value="0.370" />
-      <origin xyz="0 0 0" rpy="1.5708 0 1.5708"/>
-      <inertia ixx="1e-6" ixy="0" ixz="0" iyy="1e-6" iyz="0" izz="1e-6" />
-    </inertial>
-  </link>
-  <joint name="depth_joint" type="fixed">
-    <axis xyz="0 1 0" />
-    <origin xyz="0.165 0 1.417" rpy="0 0 0"/>
-    <parent link="base_link"/>
-    <child link="depth_link"/>
-  </joint>
-  <link name="depth_link">
-    <collision>
-      <origin xyz="0 0 0" rpy="1.3090 0 1.5708"/>
-      <geometry>
-        <mesh filename="package://telemarketing_description/meshes/depth_camera.stl" scale="0.010335 0.010335 0.010335"/>
-      </geometry>
-    </collision>
-    <visual>
-      <origin xyz="0 0 0" rpy="1.3090 0 1.5708"/>
-      <geometry>
-        <mesh filename="package://telemarketing_description/meshes/depth_camera.stl" scale="0.010335 0.010335 0.010335"/>
-      </geometry>
-      <material name="grey"/>
-    </visual>
-    <inertial>
-      <mass value="1e-5" />
-      <origin xyz="0 0 0" rpy="0 0 0"/>
-      <inertia ixx="1e-6" ixy="0" ixz="0" iyy="1e-6" iyz="0" izz="1e-6" />
-    </inertial>
-  </link>
-  <joint name="depth_optical_joint" type="fixed">
-    <origin xyz="0 0 0" rpy="-1.5708 0 -1.5708"/>
-    <parent link="depth_link"/>
-    <child link="depth_optical_link"/>
-  </joint>
-  <link name="depth_optical_link"/>
+<robot name="telemarketing" xmlns:xacro="http://www.ros.org/wiki/xacro">
+<xacro:include filename="$(find telemarketing_description)/urdf/materials.xacro" />
+<xacro:include filename="$(find telemarketing_description)/urdf/telemarketing.trans" />
+<xacro:include filename="$(find telemarketing_description)/urdf/telemarketing.gazebo" />
+<link name="base_footprint"/>
+<joint name="base_joint" type="fixed">
+  <parent link="base_footprint"/>
+  <child link="base_link"/>
+  <origin xyz="0.0 0.0 0.010" rpy="0 0 0"/>
+</joint>
+<link name="base_link">
+  <inertial>
+    <origin xyz="-0.01582626281068255 0.009388301039198908 0.44638888098941787" rpy="0 0 0"/>
+    <mass value="46.607412382470756"/>
+    <inertia ixx="12.436477" iyy="12.532565" izz="1.513354" ixy="-0.016849" iyz="-0.015147" ixz="-0.779216"/>
+  </inertial>
+  <visual>
+    <origin xyz="0 0 0" rpy="0 0 0"/>
+    <geometry>
+      <mesh filename="package://telemarketing_description/meshes/base_link.stl" scale="0.001 0.001 0.001"/>
+    </geometry>
+    <material name="silver_default"/>
+  </visual>
+  <collision>
+    <origin xyz="0 0 0.15" rpy="0 0 0"/>
+    <geometry>
+      <box size="0.64 0.64 0.2"/>
+    </geometry>
+  </collision>
+</link>
+<link name="ur_caster_1">
+  <inertial>
+    <origin xyz="-0.013500301733120085 0.001981288366912748 -0.03169998393160654" rpy="0 0 0"/>
+    <mass value="0.17193166725129566"/>
+    <inertia ixx="7.6e-05" iyy="7.9e-05" izz="6.9e-05" ixy="-0.0" iyz="-1e-05" ixz="-0.0"/>
+  </inertial>
+  <visual>
+    <origin xyz="-0.187574 0.182783 -0.062266" rpy="0 0 0"/>
+    <geometry>
+      <mesh filename="package://telemarketing_description/meshes/ur_caster_1.stl" scale="0.001 0.001 0.001"/>
+    </geometry>
+    <material name="silver_default"/>
+  </visual>
+  <collision>
+    <origin xyz="-0.02 -0.002 -0.038" rpy="0 1.5708 0"/>
+    <geometry>
+      <cylinder length="0.05" radius="0.025"/>
+    </geometry>
+  </collision>
+</link>
+<link name="br_caster_1">
+  <inertial>
+    <origin xyz="-0.013500301733128883 0.001981288366923961 -0.03169998393161214" rpy="0 0 0"/>
+    <mass value="0.17193166725129566"/>
+    <inertia ixx="7.6e-05" iyy="7.9e-05" izz="6.9e-05" ixy="-0.0" iyz="-1e-05" ixz="-0.0"/>
+  </inertial>
+  <visual>
+    <origin xyz="0.164426 0.182783 -0.062266" rpy="0 0 0"/>
+    <geometry>
+      <mesh filename="package://telemarketing_description/meshes/br_caster_1.stl" scale="0.001 0.001 0.001"/>
+    </geometry>
+    <material name="silver_default"/>
+  </visual>
+  <collision>
+    <origin xyz="-0.02 -0.002 -0.038" rpy="0 1.5708 0"/>
+    <geometry>
+      <cylinder length="0.05" radius="0.025"/>
+    </geometry>
+  </collision>
+</link>
+<link name="lidar_1">
+  <inertial>
+    <origin xyz="-0.00024518499825737505 -4.4098690871012536e-07 0.019173061203674013" rpy="0 0 0"/>
+    <mass value="0.44874442633887374"/>
+    <inertia ixx="0.000208" iyy="0.000205" izz="0.000295" ixy="0.0" iyz="0.0" ixz="1e-06"/>
+  </inertial>
+  <visual>
+    <origin xyz="-0.17441 -0.010703 -0.348266" rpy="0 0 0"/>
+    <geometry>
+      <mesh filename="package://telemarketing_description/meshes/lidar_1.stl" scale="0.001 0.001 0.001"/>
+    </geometry>
+    <material name="silver_default"/>
+  </visual>
+  <collision>
+    <origin xyz="0 0 0.02" rpy="0 0 0"/>
+    <geometry>
+      <cylinder length="0.04" radius="0.04"/>
+    </geometry>
+  </collision>
+</link>
+<link name="lwheel_1">
+  <inertial>
+    <origin xyz="2.3484289615694973e-07 -0.020637673074518137 -2.649612852456684e-07" rpy="0 0 0"/>
+    <mass value="2.17648405302028"/>
+    <inertia ixx="0.006799" iyy="0.013191" izz="0.006799" ixy="-0.0" iyz="0.0" ixz="-0.0"/>
+  </inertial>
+  <visual>
+    <origin xyz="0.002351 -0.203581 -0.100116" rpy="0 0 0"/>
+    <geometry>
+      <mesh filename="package://telemarketing_description/meshes/rwheel_1.stl" scale="0.001 0.001 0.001"/>
+    </geometry>
+    <material name="silver_default"/>
+  </visual>
+  <collision>
+    <origin xyz="0 -0.02 0" rpy="1.5708 0 0"/>
+    <geometry>
+      <cylinder length="0.04" radius="0.101"/>
+    </geometry>
+  </collision>
+</link>
+<link name="rwheel_1">
+  <inertial>
+    <origin xyz="2.3448188038715373e-07 0.02063732699882273 -2.6520921700412536e-07" rpy="0 0 0"/>
+    <mass value="2.176484032133544"/>
+    <inertia ixx="0.006799" iyy="0.013191" izz="0.006799" ixy="-0.0" iyz="-0.0" ixz="0.0"/>
+  </inertial>
+  <visual>
+    <origin xyz="0.002351 0.187147 -0.100116" rpy="0 0 0"/>
+    <geometry>
+      <mesh filename="package://telemarketing_description/meshes/lwheel_1.stl" scale="0.001 0.001 0.001"/>
+    </geometry>
+    <material name="silver_default"/>
+  </visual>
+  <collision>
+    <origin xyz="0 0.02 0" rpy="1.5708 0 0"/>
+    <geometry>
+      <cylinder length="0.04" radius="0.101"/>
+    </geometry>
+  </collision>
+</link>
+<link name="real_sense_1">
+  <inertial>
+    <origin xyz="-0.012419790832103733 -0.031108525619316624 -0.004151097658603442" rpy="0 0 0"/>
+    <mass value="0.03621223064538649"/>
+    <inertia ixx="2.3e-05" iyy="3e-06" izz="2.3e-05" ixy="0.0" iyz="0.0" ixz="-0.0"/>
+  </inertial>
+  <visual>
+    <origin xyz="-0.247213 -0.044075 -0.587532" rpy="0 0 0"/>
+    <geometry>
+      <mesh filename="package://telemarketing_description/meshes/real_sense_1.stl" scale="0.001 0.001 0.001"/>
+    </geometry>
+    <material name="silver_default"/>
+  </visual>
+  <collision>
+    <origin xyz="-0.247213 -0.044075 -0.587532" rpy="0 0 0"/>
+    <geometry>
+      <mesh filename="package://telemarketing_description/meshes/real_sense_1.stl" scale="0.001 0.001 0.001"/>
+    </geometry>
+  </collision>
+</link>
+<joint name="realsense_change" type="fixed">
+    <origin xyz="0.1 0 0" rpy="0 0 0"/>
+    <parent link="real_sense_1"/>
+    <child link="realsense_change_frame"/>
+</joint>
+<link name="realsense_change_frame"/>
+<link name="monitor1_1">
+  <inertial>
+    <origin xyz="0.06578759810161444 -0.01804654339422243 -2.6549572273992794e-07" rpy="0 0 0"/>
+    <mass value="19.65717622219914"/>
+    <inertia ixx="1.169049" iyy="0.903033" izz="0.279972" ixy="-0.007106" iyz="-1e-06" ixz="-0.0"/>
+  </inertial>
+  <visual>
+    <origin xyz="-0.030574 -0.010717 -1.090271" rpy="0 0 0"/>
+    <geometry>
+      <mesh filename="package://telemarketing_description/meshes/monitor1_1.stl" scale="0.001 0.001 0.001"/>
+    </geometry>
+    <material name="silver_default"/>
+  </visual>
+  <collision>
+    <origin xyz="-0.030574 -0.010717 -1.090271" rpy="0 0 0"/>
+    <geometry>
+      <mesh filename="package://telemarketing_description/meshes/monitor1_1.stl" scale="0.001 0.001 0.001"/>
+    </geometry>
+  </collision>
+</link>
+<link name="monitor2_1">
+  <inertial>
+    <origin xyz="0.0039472962291229735 -1.7301517323507765e-07 0.011109558387593976" rpy="0 0 0"/>
+    <mass value="1.087331660982632"/>
+    <inertia ixx="0.018585" iyy="0.005499" izz="0.01344" ixy="0.0" iyz="-0.0" ixz="0.000935"/>
+  </inertial>
+  <visual>
+    <origin xyz="-0.118841 -0.010717 -1.663148" rpy="0 0 0"/>
+    <geometry>
+      <mesh filename="package://telemarketing_description/meshes/monitor2_1.stl" scale="0.001 0.001 0.001"/>
+    </geometry>
+    <material name="silver_default"/>
+  </visual>
+  <collision>
+    <origin xyz="-0.118841 -0.010717 -1.663148" rpy="0 0 0"/>
+    <geometry>
+      <mesh filename="package://telemarketing_description/meshes/monitor2_1.stl" scale="0.001 0.001 0.001"/>
+    </geometry>
+  </collision>
+</link>
+<link name="screen_1">
+  <inertial>
+    <origin xyz="0.0025002349962530424 -3.247109095494416e-09 -3.981949106002247e-07" rpy="0 0 0"/>
+    <mass value="7.614563000001394"/>
+    <inertia ixx="0.421393" iyy="0.316678" izz="0.105509" ixy="0.0" iyz="-0.0" ixz="0.0"/>
+  </inertial>
+  <visual>
+    <origin xyz="-0.126474 -0.018765 -1.090271" rpy="0 0 0"/>
+    <geometry>
+      <mesh filename="package://telemarketing_description/meshes/screen_1.stl" scale="0.001 0.001 0.001"/>
+    </geometry>
+    <material name="silver_default"/>
+  </visual>
+  <collision>
+    <origin xyz="-0.126474 -0.018765 -1.090271" rpy="0 0 0"/>
+    <geometry>
+      <mesh filename="package://telemarketing_description/meshes/screen_1.stl" scale="0.001 0.001 0.001"/>
+    </geometry>
+  </collision>
+</link>
+<link name="bl_caster_1">
+  <inertial>
+    <origin xyz="0.015500771725656087 0.02501836560271653 -0.03169998393161695" rpy="0 0 0"/>
+    <mass value="0.17193166725129566"/>
+    <inertia ixx="7.6e-05" iyy="7.9e-05" izz="6.9e-05" ixy="-0.0" iyz="1e-05" ixz="0.0"/>
+  </inertial>
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
Commit message: Update of description and microcontroller packages - 0.3.4

File: telemarketing_description/urdf/telemarketing.xacro (robot description, xacro)
@@ -288,5 +288,5 @@
       <mesh filename="package://telemarketing_description/meshes/ultrasonido1_1.stl" scale="0.001 0.001 0.001"/>
     </geometry>
-    <material name="silver_default"/>
+    <material name="ultrasound_default"/>
   </visual>
   <collision>
@@ -308,5 +308,5 @@
       <mesh filename="package://telemarketing_description/meshes/ultrasonido2_1.stl" scale="0.001 0.001 0.001"/>
     </geometry>
-    <material name="silver_default"/>
+    <material name="ultrasound_default"/>
   </visual>
   <collision>
@@ -334,5 +334,5 @@
       <mesh filename="package://telemarketing_description/meshes/ultrasonido3_1.stl" scale="0.001 0.001 0.001"/>
     </geometry>
-    <material name="silver_default"/>
+    <material name="ultrasound_default"/>
   </visual>
   <collision>
@@ -360,5 +360,5 @@
       <mesh filename="package://telemarketing_description/meshes/ultrasonido4_1.stl" scale="0.001 0.001 0.001"/>
     </geometry>
-    <material name="silver_default"/>
+    <material name="ultrasound_default"/>
   </visual>
   <collision>
@@ -386,5 +386,5 @@
       <mesh filename="package://telemarketing_description/meshes/ultrasonido5_1.stl" scale="0.001 0.001 0.001"/>
     </geometry>
-    <material name="silver_default"/>
+    <material name="ultrasound_default"/>
   </visual>
   <collision>
@@ -412,5 +412,5 @@
       <mesh filename="package://telemarketing_description/meshes/ultrasonido6_1.stl" scale="0.001 0.001 0.001"/>
     </geometry>
-    <material name="silver_default"/>
+    <material name="ultrasound_default"/>
   </visual>
   <collision>
@@ -438,5 +438,5 @@
       <mesh filename="package://telemarketing_description/meshes/ultrasonido7_1.stl" scale="0.001 0.001 0.001"/>
     </geometry>
-    <material name="silver_default"/>
+    <material name="ultrasound_default"/>
   </visual>
   <collision>
@@ -464,5 +464,5 @@
       <mesh filename="package://telemarketing_description/meshes/ultrasonido8_1.stl" scale="0.001 0.001 0.001"/>
     </geometry>
-    <material name="silver_default"/>
+    <material name="ultrasound_default"/>
   </visual>
   <collision>
@@ -518,5 +518,5 @@
       <mesh filename="package://telemarketing_description/meshes/infrarrojo1_1.stl" scale="0.001 0.001 0.001"/>
     </geometry>
-    <material name="silver_default"/>
+    <material name="infrared_default"/>
   </visual>
   <collision>
@@ -544,5 +544,5 @@
       <mesh filename="package://telemarketing_description/meshes/infrarrojo2_1.stl" scale="0.001 0.001 0.001"/>
     </geometry>
-    <material name="silver_default"/>
+    <material name="infrared_default"/>
   </visual>
   <collision>
@@ -570,5 +570,5 @@
       <mesh filename="package://telemarketing_description/meshes/infrarrojo3_1.stl" scale="0.001 0.001 0.001"/>
     </geometry>
-    <material name="silver_default"/>
+    <material name="infrared_default"/>
   </visual>
   <collision>
@@ -596,5 +596,5 @@
       <mesh filename="package://telemarketing_description/meshes/infrarrojo4_1.stl" scale="0.001 0.001 0.001"/>
     </geometry>
-    <material name="silver_default"/>
+    <material name="infrared_default"/>
   </visual>
   <collision>
@@ -622,5 +622,5 @@
       <mesh filename="package://telemarketing_description/meshes/infrarrojo5_1.stl" scale="0.001 0.001 0.001"/>
     </geometry>
-    <material name="silver_default"/>
+    <material name="infrared_default"/>
   </visual>
   <collision>
@@ -648,5 +648,5 @@
       <mesh filename="package://telemarketing_description/meshes/infrarrojo6_1.stl" scale="0.001 0.001 0.001"/>
     </geometry>
-    <material name="silver_default"/>
+    <material name="infrared_default"/>
   </visual>
   <collision>
@@ -674,5 +674,5 @@
       <mesh filename="package://telemarketing_description/meshes/infrarrojo7_1.stl" scale="0.001 0.001 0.001"/>
     </geometry>
-    <material name="silver_default"/>
+    <material name="infrared_default"/>
   </visual>
   <collision>
@@ -700,5 +700,5 @@
       <mesh filename="package://telemarketing_description/meshes/infrarrojo8_1.stl" scale="0.001 0.001 0.001"/>
     </geometry>
-    <material name="silver_default"/>
+    <material name="infrared_default"/>
   </visual>
   <collision>
